Commit message: add Tactile

File: src/vendor/dg5f_s_description/urdf/dg5fs_right.urdf (robot description, URDF)
Before this commit: robot dg5fs_right, 26 links, 25 joints
Links:
- link link_1_tip: mass 0.00365660774514007 -> 0.016; geometry collision mesh filename=package://dg5f_s_description/meshes/dg5fs_right/tactile_tip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; visual mesh filename=package://dg5f_s_description/meshes/dg5fs_right/tactile_tip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
- link link_2_tip: mass 0.0036566 -> 0.016; geometry collision mesh filename=package://dg5f_s_description/meshes/dg5fs_right/tactile_tip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; visual mesh filename=package://dg5f_s_description/meshes/dg5fs_right/tactile_tip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
- link link_3_tip: mass 0.00365660774514011 -> 0.016; geometry collision mesh filename=package://dg5f_s_description/meshes/dg5fs_right/tactile_tip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; visual mesh filename=package://dg5f_s_description/meshes/dg5fs_right/tactile_tip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
- link link_4_tip: mass 0.0036566077451401 -> 0.016; geometry collision mesh filename=package://dg5f_s_description/meshes/dg5fs_right/tactile_tip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; visual mesh filename=package://dg5f_s_description/meshes/dg5fs_right/tactile_tip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
- link link_5_tip: mass 0.00365660774514004 -> 0.016; geometry collision mesh filename=package://dg5f_s_description/meshes/dg5fs_right/tactile_tip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; visual mesh filename=package://dg5f_s_description/meshes/dg5fs_right/tactile_tip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
Joints:
- joint joint_1_tip: origin xyz=0.0289 0 0 rpy=0 0 0 -> xyz=0.0259 0 0 rpy=0 0 0
- joint joint_2_tip: origin xyz=0.018 0 0 rpy=0 0 0 -> xyz=0.015 0 0 rpy=0 0 0
- joint joint_3_tip: origin xyz=0.018 0 0 rpy=0 0 0 -> xyz=0.015 0 0 rpy=0 0 0
- joint joint_4_tip: origin xyz=0.018 0 0 rpy=0 0 0 -> xyz=0.015 0 0 rpy=0 0 0
- joint joint_5_tip: origin xyz=0.0289 0 0 rpy=0 0 0 -> xyz=0.0259 0 0 rpy=0 0 0

File: src/vendor/dg5f_s_description/urdf/dg5fs_right_w_mount.urdf (robot description, URDF)
Before this commit: robot dg5fs_right, 27 links, 26 joints
Links:
- link link_1_tip: mass 0.00365660774514007 -> 0.016; geometry collision mesh filename=package://dg5f_s_description/meshes/dg5fs_right/tactile_tip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; visual mesh filename=package://dg5f_s_description/meshes/dg5fs_right/tactile_tip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
- link link_2_tip: mass 0.0036566 -> 0.016; geometry collision mesh filename=package://dg5f_s_description/meshes/dg5fs_right/tactile_tip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; visual mesh filename=package://dg5f_s_description/meshes/dg5fs_right/tactile_tip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
- link link_3_tip: mass 0.00365660774514011 -> 0.016; geometry collision mesh filename=package://dg5f_s_description/meshes/dg5fs_right/tactile_tip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; visual mesh filename=package://dg5f_s_description/meshes/dg5fs_right/tactile_tip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
- link link_4_tip: mass 0.0036566077451401 -> 0.016; geometry collision mesh filename=package://dg5f_s_description/meshes/dg5fs_right/tactile_tip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; visual mesh filename=package://dg5f_s_description/meshes/dg5fs_right/tactile_tip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
- link link_5_tip: mass 0.00365660774514004 -> 0.016; geometry collision mesh filename=package://dg5f_s_description/meshes/dg5fs_right/tactile_tip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; visual mesh filename=package://dg5f_s_description/meshes/dg5fs_right/tactile_tip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
Joints:
- joint joint_1_tip: origin xyz=0.0289 0 0 rpy=0 0 0 -> xyz=0.0259 0 0 rpy=0 0 0
- joint joint_2_tip: origin xyz=0.018 0 0 rpy=0 0 0 -> xyz=0.015 0 0 rpy=0 0 0
- joint joint_3_tip: origin xyz=0.018 0 0 rpy=0 0 0 -> xyz=0.015 0 0 rpy=0 0 0
- joint joint_4_tip: origin xyz=0.018 0 0 rpy=0 0 0 -> xyz=0.015 0 0 rpy=0 0 0
- joint joint_5_tip: origin xyz=0.0289 0 0 rpy=0 0 0 -> xyz=0.0259 0 0 rpy=0 0 0
