Commit message: 0902

File: src/vendor/dg5f_s_description/urdf/dg5fs_15dof_right.urdf (robot description, URDF)
Before this commit: robot dg5fs_right, 21 links, 20 joints
Joints:
- joint joint_1_1: limit lower=-1.5707963267948966 upper=1.5707963267948966 effort=7.5 velocity=3.141592653589793 -> lower=-0.2792526803190927 upper=0.9250245035569946 effort=7.5 velocity=3.141592653589793
- joint joint_1_2: limit lower=-2.670353755551324 upper=0 effort=7.5 velocity=3.141592653589793 -> lower=-1.8500490071139892 upper=0 effort=7.5 velocity=3.141592653589793

File: src/vendor/dg5f_s_description/urdf/dg5fs_15dof_right_w_mount.urdf (robot description, URDF)
Before this commit: robot dg5fs_right, 22 links, 21 joints
Joints:
- joint joint_1_1: limit lower=-1.5707963267948966 upper=1.5707963267948966 effort=7.5 velocity=3.141592653589793 -> lower=-0.2792526803190927 upper=0.9250245035569946 effort=7.5 velocity=3.141592653589793
- joint joint_1_2: limit lower=-2.670353755551324 upper=0 effort=7.5 velocity=3.141592653589793 -> lower=-1.8500490071139892 upper=0 effort=7.5 velocity=3.141592653589793

File: src/vendor/dg5f_s_description/urdf/dg5fs_right.urdf (robot description, URDF)
Before this commit: robot dg5fs_right, 26 links, 25 joints
Joints:
- joint joint_1_1: limit lower=-1.5707963267948966 upper=1.5707963267948966 effort=7.5 velocity=3.141592653589793 -> lower=-0.2792526803190927 upper=0.9250245035569946 effort=7.5 velocity=3.141592653589793
- joint joint_1_2: limit lower=-2.670353755551324 upper=0 effort=7.5 velocity=3.141592653589793 -> lower=-1.8500490071139892 upper=0 effort=7.5 velocity=3.141592653589793

File: src/vendor/dg5f_s_description/urdf/dg5fs_right_w_mount.urdf (robot description, URDF)
Before this commit: robot dg5fs_right, 27 links, 26 joints
Joints:
- joint joint_1_1: limit lower=-1.5707963267948966 upper=1.5707963267948966 effort=7.5 velocity=3.141592653589793 -> lower=-0.2792526803190927 upper=0.9250245035569946 effort=7.5 velocity=3.141592653589793
- joint joint_1_2: limit lower=-2.670353755551324 upper=0 effort=7.5 velocity=3.141592653589793 -> lower=-1.8500490071139892 upper=0 effort=7.5 velocity=3.141592653589793
